Commit message: tested and fixed drvietrain code

File: arm/urdf/Arm.urdf (robot description, URDF)
Before this commit: robot Arm, 5 links, 4 joints
Links:
- link base_link: mass None -> 5; geometry collision box size=0.23741888 0.07387082 0.01; visual box size=0.23741888 0.07387082 0.01
- link bicep: mass None -> 5; geometry collision box size=0.03556 0.0766826 0.1439164; visual box size=0.03556 0.0766826 0.1439164
- link end_effector: mass None -> 5; geometry collision box size=0.0673354 0.1293368 0.1192022; visual box size=0.0673354 0.1293368 0.1192022
- link forearm: mass None -> 5; geometry collision box size=0.03556 0.0701802 0.1613662; visual box size=0.03556 0.0701802 0.1613662
- link socket: mass None -> 5; geometry collision cylinder length=0.0508 radius=0.0127; visual cylinder length=0.0508 radius=0.0127
