Commit message: added new arm ik config

File: arm/urdf/Arm_gazebo.urdf (robot description, URDF)
Before this commit: robot Arm, 5 links, 4 joints
Links:
- removed link bicep
- removed link end_effector
- removed link forearm
- removed link socket
- added link link_claw, mass 0; collision mesh filename=package://urdf_tutorial/right-arm/dc12_a01_spacer_ring.stl; collision mesh filename=package://urdf_tutorial/right-arm/dc12_a01_spacer_ring.stl
- added link link_elbow, mass 0; collision mesh filename=package://urdf_tutorial/right-arm/10-32_x_0.75in_buttonhead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; collision mesh filename=package://urdf_tutorial/right-arm/10-32_x_0.75in_buttonhead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
- added link link_forearm, mass 0; collision mesh filename=package://urdf_tutorial/right-arm/10-32_x_0.75in_buttonhead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; collision mesh filename=package://urdf_tutorial/right-arm/10-32_x_0.75in_buttonhead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
- added link link_socket, mass 0; collision mesh filename=package://urdf_tutorial/right-arm/.5_hexbearing_1.125_od.stl; collision mesh filename=package://urdf_tutorial/right-arm/.5_hexbearing_1.125_od.stl
- link base_link: mass None -> 0; geometry collision mesh filename=package://urdf_tutorial/right-arm/.5_hexbearing_1.125_od.stl; collision mesh filename=package://urdf_tutorial/right-arm/.5_hexbearing_1.125_od.stl
Joints:
- joint elbow: axis 0 1 0 -> 0 0 1; child forearm -> link_forearm; origin xyz=0 0 0.1439164 rpy=0 0 0 -> xyz=0.166399 -0.0715838 -0.0251898 rpy=-1.66708e-14 -1.48395e-14 1.16453; parent bicep -> link_elbow
- joint shoulder_pitch: axis 0 1 0 -> 0 0 1; child bicep -> link_elbow; origin xyz=0 0.0141986 0.0254 rpy=0 0 0 -> xyz=-0.0297467 -2.91434e-16 -0.0893164 rpy=1.5708 0.960485 1.5708; parent socket -> link_socket
- joint shoulder_yaw: child socket -> link_socket; limit (none) -> effort=1 velocity=20; origin xyz=0.10600944 0 0.0303 rpy=0 0 0 -> xyz=-0.050972 -0.0908091 -0.0376234 rpy=3.14159 -4.29356e-16 2.5501
- joint wrist: child end_effector -> link_claw; limit (none) -> effort=1 velocity=20; origin xyz=0 0 0.1613662 rpy=0 0 0 -> xyz=4.16334e-16 -0.178438 0.03 rpy=-1.5708 1.5708 0; parent forearm -> link_forearm
