Commit message: move it servo working with new config

File: right_arm_urdf/urdf/robot.urdf (robot description, URDF)
Before this commit: robot jacker, 5 links, 4 joints
Links:
- link base_link: mass 5 -> 20
- link link_claw: mass 5 -> 0.5
- link link_elbow: mass 5 -> 0.5
- link link_forearm: mass 5 -> 0.5
- link link_socket: mass 5 -> 0.5
